File: core.kicad_sch (KiCad schematic)
At the start: 41 parts, among them U1 ESP32-P4, U2 W25Q128JVS, Y1 40MHz 10ppm, Y2 32.768k

Commit message: Finish off schematic
Parts:
- U1: footprint Espressif:ESP32-P4 -> PCM_Espressif:ESP32-P4
Connections:
- net GPIO0 renamed IO0/LSE
- net IO0/LSE: no longer U1.104 (GPIO0/ADC)
- net GPIO1 renamed IO1/LSE
- net GPIO10 renamed IO10/TDO
- net GPIO11 renamed IO11/nRST
- net GPIO12 renamed IO12
- net GPIO13 renamed IO13
- net GPIO14 renamed IO14/UART_TX
- net GPIO15 renamed IO15/UART_RX
- net GPIO16: no longer names the net of U1.17 (GPIO16/ADC)
- net GPIO17: no longer names the net of U1.18 (GPIO17/ADC)
- net GPIO18: no longer names the net of U1.19 (GPIO18/ADC)
- net GPIO19: no longer names the net of U1.20 (GPIO19/ADC)
- net GPIO2: no longer names the net of U1.2 (GPIO2/ADC)
- net GPIO20: no longer names the net of U1.22 (GPIO20/ADC)
- net GPIO21: no longer names the net of U1.23 (GPIO21/ADC)
- net GPIO22: no longer names the net of U1.24 (GPIO22/ADC)
- net GPIO23: no longer names the net of U1.25 (GPIO23/ADC)
- net GPIO24 renamed IO24/JTAG_DM
- net GPIO25 renamed IO25/JTAG_DP
- net GPIO3: no longer names the net of U1.3 (GPIO3/ADC)
- net GPIO35/BOOT renamed IO35/BOOT
- net GPIO37/U0TXD renamed IO37/U0TXD
- net GPIO38/U0RXD renamed IO38/U0RXD
- net GPIO39 renamed IO39/SDDAT0
- net GPIO4 renamed IO4/TRST
- net GPIO40 renamed IO40/SDDAT1
- net GPIO41 renamed IO41/SDDAT2
- net GPIO42 renamed IO42/SDDAT3
- net GPIO43 renamed IO43/SDCLK
- net GPIO44 renamed IO44/SDCMD
- net GPIO45 renamed IO45/SDDET
- net GPIO46: no longer names the net of U1.88 (GPIO46)
- net GPIO47: no longer names the net of U1.89 (GPIO47)
- net GPIO48: no longer names the net of U1.90 (GPIO48)
- net GPIO49: no longer names the net of U1.92 (GPIO49/ADC)
- net GPIO5 renamed IO5/TDI
- net GPIO50: no longer names the net of U1.93 (GPIO50/ADC)
- net GPIO51: no longer names the net of U1.94 (GPIO51/ADC)
- net GPIO52: no longer names the net of U1.95 (GPIO52/ADC)
- net GPIO53: no longer names the net of U1.97 (GPIO53/ADC)
- net GPIO54: no longer names the net of U1.98 (GPIO54/ADC)
- net GPIO6 renamed IO6/SWDIO
- net GPIO7 renamed IO7/SWCLK
- net GPIO8 renamed IO8/BOOT
- net GPIO9 renamed IO9/nRST
- new net IO0/LSE1: U1.104 (GPIO0/ADC)
- no-connect marks 24 -> 43
Other:
- company: (none) -> By Jackson Ming Hu <huming2207@gmail.com> Copright (C) 2025 
- title: (none) -> Soul Probe
- moved on the sheet: C20, C21, C32, C33, C34, C8

Commit message: Typo fix
Parts:
- U1: footprint PCM_Espressif:ESP32-P4 -> Espressif:ESP32-P4
Connections:
- net IO0/LSE1 is gone; now on net IO0/LSE: U1.104 (GPIO0/ADC)
Changed lines of the file:
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@@
 		)
 	)
-	(global_label "IO0{slash}LSE1"
+	(global_label "IO0{slash}LSE"
 		(shape input)
 		(at 144.78 96.52 90)
@@
 		)
 		(property "Intersheetrefs" "${INTERSHEET_REFS}"
-			(at 144.78 87.85 90)
+			(at 144.78 85.6729 90)
 			(effects
 				(font
@@
 			)
 		)
-		(property "Footprint" "PCM_Espressif:ESP32-P4"
+		(property "Footprint" "Espressif:ESP32-P4"
 			(at 121.92 185.42 0)
 			(effects

Commit message: Assign footprint
Parts:
- C11, C14, C17, C18, C19, C20, C22, C27, C28, C30, C34: footprint Capacitor_SMD:C_0603_1608Metric -> Capacitor_SMD:C_0402_1005Metric
Changed lines of the file:
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@@
 			)
 		)
-		(property "Footprint" "Capacitor_SMD:C_0603_1608Metric"
+		(property "Footprint" "Capacitor_SMD:C_0402_1005Metric"
 			(at 336.2452 96.52 0)
 			(effects
@@
 			)
 		)
-		(property "Footprint" "Capacitor_SMD:C_0603_1608Metric"
+		(property "Footprint" "Capacitor_SMD:C_0402_1005Metric"
 			(at 101.2952 184.15 0)
 			(effects
@@
 			)
 		)
-		(property "Footprint" "Capacitor_SMD:C_0603_1608Metric"
+		(property "Footprint" "Capacitor_SMD:C_0402_1005Metric"
 			(at 116.5352 93.98 0)
 			(effects
@@
 			)
 		)
-		(property "Footprint" "Capacitor_SMD:C_0603_1608Metric"
+		(property "Footprint" "Capacitor_SMD:C_0402_1005Metric"
 			(at 319.7352 96.52 0)
 			(effects
@@
 			)
 		)
-		(property "Footprint" "Capacitor_SMD:C_0603_1608Metric"
+		(property "Footprint" "Capacitor_SMD:C_0402_1005Metric"
 			(at 267.6652 167.64 0)
 			(effects
@@
 			)
 		)
-		(property "Footprint" "Capacitor_SMD:C_0603_1608Metric"
+		(property "Footprint" "Capacitor_SMD:C_0402_1005Metric"
 			(at 82.2452 140.97 0)
 			(effects
@@
 			)
 		)
-		(property "Footprint" "Capacitor_SMD:C_0603_1608Metric"
+		(property "Footprint" "Capacitor_SMD:C_0402_1005Metric"
 			(at 270.2052 96.52 0)
 			(effects
@@
 			)
 		)
-		(property "Footprint" "Capacitor_SMD:C_0603_1608Metric"
+		(property "Footprint" "Capacitor_SMD:C_0402_1005Metric"
 			(at 357.8352 96.52 0)
 			(effects
@@
 			)
 		)
-		(property "Footprint" "Capacitor_SMD:C_0603_1608Metric"
+		(property "Footprint" "Capacitor_SMD:C_0402_1005Metric"
 			(at 347.6752 96.52 0)
 			(effects
@@
 			)
 		)
-		(property "Footprint" "Capacitor_SMD:C_0603_1608Metric"
+		(property "Footprint" "Capacitor_SMD:C_0402_1005Metric"
 			(at 265.1252 223.52 0)
 			(effects
@@
 			)
 		)
-		(property "Footprint" "Capacitor_SMD:C_0603_1608Metric"
+		(property "Footprint" "Capacitor_SMD:C_0402_1005Metric"
 			(at 120.3452 214.63 0)
 			(effects

Commit message: Refine footprint matching
Parts:
- removed U2: W25Q128JVS, Package_SO:SOIC-8_5.3x5.3mm_P1.27mm, symbol Memory_Flash:W25Q128JVS
- added U5: W25Q128JVE, Package_SON:WSON-8-1EP_8x6mm_P1.27mm_EP3.4x4.3mm, symbol Memory_Flash:W25Q128JVE
Connections:
- net FLASH_CK: now also U5.6 (CLK)
- net FLASH_CS: now also U5.1 (~{CS})
- net FLASH_D: now also U5.5 (DI/IO_{0})
- net FLASH_HD: now also U5.7 (~{HOLD}/~{RESET}/IO_{3})
- net FLASH_Q: now also U5.2 (DO/IO_{1})
- net FLASH_WP: now also U5.3 (~{WP}/IO_{2})
- net GND: now also U5.4 (GND), U5.9 (EP)
- net VDDO_FLASH: now also U5.8 (VCC)
Changed lines of the file:
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@@
 	)
 	(junction
+		(at 364.49 171.45)
+		(diameter 0)
+		(color 0 0 0 0)
+	)
+	(junction
 		(at 100.33 175.26)
 		(diameter 0)
@@
 	(wire
 		(pts
+			(xy 367.03 168.91) (xy 367.03 171.45)
+		)
+		(stroke
+			(width 0)
+			(type default)
+		)
+	)
+	(wire
+		(pts
 			(xy 116.84 129.54) (xy 119.38 129.54)
 		)
@@
 	(wire
 		(pts
+			(xy 364.49 171.45) (xy 364.49 173.99)
+		)
+		(stroke
+			(width 0)
+			(type default)
+		)
+	)
+	(wire
+		(pts
 			(xy 130.81 205.74) (xy 130.81 207.01)
 		)
@@
 	(wire
 		(pts
+			(xy 367.03 171.45) (xy 364.49 171.45)
+		)
+		(stroke
+			(width 0)
+			(type default)
+		)
+	)
+	(wire
+		(pts
 			(xy 289.56 151.13) (xy 289.56 153.67)
 		)
@@
 	(wire
 		(pts
-			(xy 364.49 168.91) (xy 364.49 173.99)
+			(xy 364.49 168.91) (xy 364.49 171.45)
 		)
 		(stroke
@@
 	)
 	(symbol
+		(lib_id "Memory_Flash:W25Q128JVE")
+		(at 364.49 156.21 0)
+		(unit 1)
+		(exclude_from_sim no)
+		(in_bom yes)
+		(on_board yes)
+		(dnp no)
+		(fields_autoplaced yes)
+		(property "Reference" "U5"
+			(at 375.92 154.9399 0)
+			(effects
+				(font
+					(size 1.27 1.27)
+				)
+				(justify left)
+			)
+		)
+		(property "Value" "W25Q128JVE"
+			(at 375.92 157.4799 0)
+			(effects
+				(font
+					(size 1.27 1.27)
+				)
+				(justify left)
+			)
+		)
+		(property "Footprint" "Package_SON:WSON-8-1EP_8x6mm_P1.27mm_EP3.4x4.3mm"
+			(at 364.49 133.35 0)
+			(effects
+				(font
+					(size 1.27 1.27)
+				)
+				(hide yes)
+			)
+		)
+		(property "Datasheet" "https://www.winbond.com/resource-files/w25q128jv_dtr%20revc%2003272018%20plus.pdf"
+			(at 364.49 130.81 0)
+			(effects
+				(font
+					(size 1.27 1.27)
+				)
+				(hide yes)
+			)
+		)
+		(property "Description" "128Mbit / 16MiB Serial Flash Memory, Standard/Dual/Quad SPI, 2.7-3.6V, WSON-8"
+			(at 364.49 128.27 0)
+			(effects
+				(font
+					(size 1.27 1.27)
+				)
+				(hide yes)
+			)
+		)
+		(pin "1"
+		)
+		(pin "6"
+		)
+		(pin "5"
+		)
+		(pin "2"
+		)
+		(pin "3"
+		)
+		(pin "7"
+		)
+		(pin "8"
+		)
+		(pin "4"
+		)
+		(pin "9"
+		)
+		(instances
+			(project ""
+				(path "/e5669c4b-5924-4e3d-8c50-ca267302db45/d98346a4-aabd-4550-99ea-ed9362dec0b9"
+					(reference "U5")
+					(unit 1)
+				)
+			)
+		)
+	)
+	(symbol
 		(lib_id "power:GND")
 		(at 218.44 95.25 0)
@@
 					(unit 1)
 				)
-			)
-		)
-	)
-	(symbol
-		(lib_id "Memory_Flash:W25Q128JVS")
-		(at 364.49 156.21 0)
-		(unit 1)
-		(exclude_from_sim no)
-		(in_bom yes)
-		(on_board yes)
-		(dnp no)
-		(fields_autoplaced yes)
-		(property "Reference" "U2"
-			(at 375.92 154.9399 0)
-			(effects
-				(font
-					(size 1.27 1.27)
-				)
-				(justify left)
-			)
-		)
-		(property "Value" "W25Q128JVS"
-			(at 375.92 157.4799 0)
-			(effects
-				(font
-					(size 1.27 1.27)
-				)
-				(justify left)
-			)
-		)
-		(property "Footprint" "Package_SO:SOIC-8_5.3x5.3mm_P1.27mm"
-			(at 364.49 133.35 0)
-			(effects
-				(font
-					(size 1.27 1.27)
-				)
-				(hide yes)
-			)
-		)
-		(property "Datasheet" "https://www.winbond.com/resource-files/w25q128jv_dtr%20revc%2003272018%20plus.pdf"
-			(at 364.49 130.81 0)
-			(effects
-				(font
-					(size 1.27 1.27)
-				)
-				(hide yes)
-			)
-		)
-		(property "Description" "128Mbit / 16MiB Serial Flash Memory, Standard/Dual/Quad SPI, 2.7-3.6V, SOIC-8"
-			(at 364.49 128.27 0)
-			(effects
-				(font
-					(size 1.27 1.27)
-				)
-				(hide yes)
-			)
-		)
-		(property "LCSC" "C97521"
-			(at 375.92 154.9399 0)
-			(effects
-				(font
-					(size 1.27 1.27)
-				)
-				(hide yes)
-			)
-		)
-		(pin "4"
-		)
-		(pin "2"
-		)
-		(pin "6"
-		)
-		(pin "5"
-		)
-		(pin "8"
-		)
-		(pin "3"
-		)
-		(pin "1"
-		)
-		(pin "7"
-		)
-		(instances
-			(project "soulprobe"
-				(path "/e5669c4b-5924-4e3d-8c50-ca267302db45/d98346a4-aabd-4550-99ea-ed9362dec0b9"
-					(reference "U2")
-					(unit 1)
-				)

Commit message: Rev 1
Connections:
- net IO2: now reaches U1.2 (GPIO2/ADC)
- net IO3: now reaches U1.3 (GPIO3/ADC)
- net IO26: now reaches U1.55 (GPIO26/ADC/USB)
- net IO27: now reaches U1.56 (GPIO27/ADC/USB)
- net IO46: now reaches U1.88 (GPIO46)
- net IO47: now reaches U1.89 (GPIO47)
- net IO48: now reaches U1.90 (GPIO48)
- net IO49: now reaches U1.92 (GPIO49/ADC)
- net IO50: now reaches U1.93 (GPIO50/ADC)
- net IO51: now reaches U1.94 (GPIO51/ADC)
- net IO52: now reaches U1.95 (GPIO52/ADC)
- net IO53: now reaches U1.97 (GPIO53/ADC)
- no-connect marks 43 -> 27
Other:
- moved on the sheet: C10, C25, Y2
