File: peripheral.kicad_sch (KiCad schematic)
At the start: 24 parts, among them J1 Conn_01x26_Pin, J2 UART_PROG, J3 Micro_SD_Card_Det_Hirose_DM3AT, J4 USB_HS, J6 USB_JTAG, SW1 BOOT, SW2 RST

Commit message: Finish off schematic
Parts:
- removed J1: Conn_01x26_Pin, Connector_PinHeader_2.54mm:PinHeader_2x13_P2.54mm_Vertical, symbol Connector:Conn_01x26_Pin
- removed J4: USB_HS, Connector_USB:USB_C_Receptacle_HRO_TYPE-C-31-M-12, symbol Connector:USB_C_Receptacle_USB2.0
- removed J6: USB_JTAG, Connector_USB:USB_C_Receptacle_HRO_TYPE-C-31-M-12, symbol Connector:USB_C_Receptacle_USB2.0
- added J1: JTAG, Connector_PinHeader_2.54mm:PinHeader_2x10_P2.54mm_Vertical, symbol Connector_Generic:Conn_02x10_Odd_Even
- added J4: USB_MAIN, symbol Connector:USB_C_Receptacle_USB2.0_16P
- added J5: USB_DBG, symbol Connector:USB_C_Receptacle_USB2.0_16P
- added R5, R6: 22R, symbol Device:R
Connections:
- net +3V3: now also J1.2 (Pin_2)
- net +5V: now also J4.A4 (VBUS), J4.A9 (VBUS), J4.B4 (VBUS), J4.B9 (VBUS), J5.A4 (VBUS), J5.A9 (VBUS), J5.B4 (VBUS), J5.B9 (VBUS)
- net GND: now also J1.10 (Pin_10), J1.12 (Pin_12), J1.4 (Pin_4), J1.6 (Pin_6), J1.8 (Pin_8), J4.A1 (GND), J4.A12 (GND), J4.B1 (GND), J4.B12 (GND), J4.S1 (SHIELD), J5.A1 (GND), J5.A12 (GND), J5.B1 (GND), J5.B12 (GND), J5.S1 (SHIELD)
- net at R22.1: now also J4.A6 (D+), J4.B6 (D+)
- net at R10.1: now also J5.A5 (CC1)
- net at R9.1: now also J5.B5 (CC2)
- net at R20.1: now also J4.A5 (CC1)
- net at R21.2: now also J4.A7 (D-), J4.B7 (D-)
- net at R4.1: now also J4.B5 (CC2)
- net GPIO35/BOOT renamed IO35/BOOT
- net GPIO37/U0TXD renamed IO37/U0TXD
- net GPIO38/U0RXD renamed IO38/U0RXD
- net GPIO39 renamed IO39/SDDAT0
- net GPIO40 renamed IO40/SDDAT1
- net GPIO41 renamed IO41/SDDAT2
- net GPIO42 renamed IO42/SDDAT3
- net GPIO43 renamed IO43/SDCLK
- net GPIO44 renamed IO44/SDCMD
- net GPIO45 renamed IO45/SDDET
- new net: J1.7 (Pin_7), R5.2
- new net: J1.9 (Pin_9), R6.1
- new net +5v: J1.19 (Pin_19)
- new net IO10/TDO: J1.15 (Pin_15)
- new net IO11/nRST: J1.17 (Pin_17)
- new net IO12: J1.14 (Pin_14)
- new net IO13: J1.16 (Pin_16)
- new net IO14/UART_TX: J1.18 (Pin_18)
- new net IO15/UART_RX: J1.20 (Pin_20)
- new net IO24/JTAG_DM: J5.A7 (D-), J5.B7 (D-)
- new net IO25/JTAG_DP: J5.A6 (D+), J5.B6 (D+)
- new net IO4/TRST: J1.3 (Pin_3)
- new net IO5/TDI: J1.5 (Pin_5)
- new net IO6/SWDIO: R5.1
- new net IO7/SWCLK: R6.2
- new net IO8/BOOT: J1.11 (Pin_11)
- new net IO9/nRST: J1.13 (Pin_13)
- no-connect marks 4 -> 5
Other:
- company: (none) -> By Jackson Ming Hu <huming2207@gmail.com> Copright (C) 2025 
- title: (none) -> Soul Probe
- moved on the sheet: C35, C36, R2, R3, SW1, SW2

Commit message: Typo fix
Connections:
- net +5v is gone; now on net +5V: J1.19 (Pin_19)
Changed lines of the file:
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@@
 			)
 		)
-		(property "Value" "+5v"
+		(property "Value" "+5V"
 			(at 221.996 133.35 0)
 			(effects

Commit message: Assign footprint
Parts:
- J4, J5: footprint (none) -> Connector_USB:USB_C_Receptacle_HRO_TYPE-C-31-M-12
- R5, R6: footprint (none) -> Resistor_SMD:R_0402_1005Metric
Changed lines of the file:
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@@
 			)
 		)
-		(property "Footprint" ""
+		(property "Footprint" "Resistor_SMD:R_0402_1005Metric"
 			(at 219.71 124.968 90)
 			(effects
@@
 			)
 		)
-		(property "Footprint" ""
+		(property "Footprint" "Connector_USB:USB_C_Receptacle_HRO_TYPE-C-31-M-12"
 			(at 52.07 147.32 0)
 			(effects
@@
 			)
 		)
-		(property "Footprint" ""
+		(property "Footprint" "Resistor_SMD:R_0402_1005Metric"
 			(at 219.71 123.952 90)
 			(effects
@@
 			)
 		)
-		(property "Footprint" ""
+		(property "Footprint" "Connector_USB:USB_C_Receptacle_HRO_TYPE-C-31-M-12"
 			(at 181.61 63.5 0)
 			(effects

Commit message: Refine footprint matching
Parts:
- removed J5: USB_DBG, Connector_USB:USB_C_Receptacle_HRO_TYPE-C-31-M-12, symbol Connector:USB_C_Receptacle_USB2.0_16P
- removed R10, R9: 5.11k, Resistor_SMD:R_0402_1005Metric, symbol Device:R_Small
- added J5: USB_DBG, Connector_PinSocket_1.27mm:PinSocket_1x04_P1.27mm_Vertical, symbol Connector:Conn_01x04_Pin
Connections:
- net +5V: now also J5.1 (Pin_1)
- net GND: now also J5.4 (Pin_4)
- net IO24/JTAG_DM: now also J5.2 (Pin_2)
- net IO25/JTAG_DP: now also J5.3 (Pin_3)
- no-connect marks 5 -> 3

Commit message: Rev 1
Parts:
- removed J1: JTAG, Connector_PinHeader_2.54mm:PinHeader_2x10_P2.54mm_Vertical, symbol Connector_Generic:Conn_02x10_Odd_Even
- removed J3: Micro_SD_Card_Det_Hirose_DM3AT, Connector_Card:microSD_HC_Hirose_DM3AT-SF-PEJM5, symbol Connector:Micro_SD_Card_Det_Hirose_DM3AT
- removed J4: USB_MAIN, Connector_USB:USB_C_Receptacle_HRO_TYPE-C-31-M-12, symbol Connector:USB_C_Receptacle_USB2.0_16P
- removed R13, R14, R15, R16, R17, R18, R19: 10k, Resistor_SMD:R_0402_1005Metric, symbol Device:R
- removed R20, R4: 5.11k, Resistor_SMD:R_0402_1005Metric, symbol Device:R_Small
- removed R21, R22: 0R, Resistor_SMD:R_0402_1005Metric, symbol Device:R_Small
- removed R5, R6: 22R, Resistor_SMD:R_0402_1005Metric, symbol Device:R
- added C1, C3: 22uF, Capacitor_SMD:C_0402_1005Metric, symbol Device:C
- added J1: PROG_PINS, Connector_PinHeader_1.27mm:PinHeader_2x10_P1.27mm_Vertical_SMD, symbol Connector_Generic:Conn_02x10_Row_Letter_First
- added J3: DBG_PINS, Connector_PinHeader_1.27mm:PinHeader_2x10_P1.27mm_Vertical_SMD, symbol Connector_Generic:Conn_02x10_Row_Letter_First
- added J4: SDIO_PINS, Connector_PinHeader_1.27mm:PinHeader_2x10_P1.27mm_Vertical_SMD, symbol Connector_Generic:Conn_02x10_Row_Letter_First
- added L1: 2.2uH/3A, Inductor_SMD:L_Changjiang_FTC322510S, symbol Device:L
- added U3: TLV62569DBV, Package_TO_SOT_SMD:SOT-23-5, symbol Regulator_Switching:TLV62569DBV
- J2: footprint Connector_PinHeader_2.54mm:PinHeader_1x06_P2.54mm_Vertical -> Connector_PinHeader_1.27mm:PinHeader_1x06_P1.27mm_Vertical
Connections:
- net +3V3: now also C1.1, J1.a1 (Pin_a1), J1.b1 (Pin_b1), J3.a1 (Pin_a1), J3.a2 (Pin_a2), J3.b1 (Pin_b1), J3.b2 (Pin_b2), J4.a1 (Pin_a1), J4.b1 (Pin_b1), U3.4 (VIN)
- net CHIP_PU: now also J3.a3 (Pin_a3)
- net GND: now also C1.2, C3.2, J1.a7 (Pin_a7), J1.b2 (Pin_b2), J1.b6 (Pin_b6), J1.b8 (Pin_b8), J3.a10 (Pin_a10), J3.a5 (Pin_a5), J3.a9 (Pin_a9), J3.b10 (Pin_b10), J3.b9 (Pin_b9), J4.a10 (Pin_a10), J4.b10 (Pin_b10), U3.2 (GND)
- net IO10/TDO: now also J1.a9 (Pin_a9)
- net IO11/nRST: now also J1.a10 (Pin_a10)
- net IO12: now also J1.b5 (Pin_b5)
- net IO13: now also J1.b7 (Pin_b7)
- net IO14/UART_TX: now also J1.b9 (Pin_b9)
- net IO15/UART_RX: now also J1.b10 (Pin_b10)
- net IO24/JTAG_DM: now also J3.b6 (Pin_b6)
- net IO25/JTAG_DP: now also J3.b5 (Pin_b5)
- net IO35/BOOT: now also J3.a4 (Pin_a4)
- net IO37/U0TXD: now also J3.a7 (Pin_a7)
- net IO38/U0RXD: now also J3.a6 (Pin_a6)
- net IO39/SDDAT0: now also J4.a3 (Pin_a3)
- net IO40/SDDAT1: now also J4.a4 (Pin_a4)
- net IO41/SDDAT2: now also J4.a5 (Pin_a5)
- net IO42/SDDAT3: now also J4.a6 (Pin_a6)
- net IO43/SDCLK: now also J4.a7 (Pin_a7)
- net IO44/SDCMD: now also J4.a8 (Pin_a8)
- net IO45/SDDET: now also J4.a9 (Pin_a9)
- net IO4/TRST: now also J1.a2 (Pin_a2)
- net IO5/TDI: now also J1.a3 (Pin_a3)
- net IO6/SWDIO: now also J1.a4 (Pin_a4)
- net IO7/SWCLK: now also J1.a5 (Pin_a5)
- net IO8/BOOT: now also J1.a6 (Pin_a6)
- net IO9/nRST: now also J1.a8 (Pin_a8)
- net USB_DM: now also J3.b8 (Pin_b8)
- net USB_DP: now also J3.b7 (Pin_b7)
- new net: L1.1, U3.3 (SW)
- new net +1V2: C3.1, L1.2
- new net EN_DCDC: J4.a2 (Pin_a2), U3.1 (EN)
- new net FB_DCDC: U3.5 (FB)
- new net IO2: J1.b3 (Pin_b3)
- new net IO26: J3.b4 (Pin_b4)
- new net IO27: J3.b3 (Pin_b3)
- new net IO3: J1.b4 (Pin_b4)
- new net IO46: J4.b2 (Pin_b2)
- new net IO47: J4.b3 (Pin_b3)
- new net IO48: J4.b4 (Pin_b4)
- new net IO49: J4.b5 (Pin_b5)
- new net IO50: J4.b6 (Pin_b6)
- new net IO51: J4.b7 (Pin_b7)
- new net IO52: J4.b8 (Pin_b8)
- new net IO53: J4.b9 (Pin_b9)
- no-connect marks 3 -> 1
Other:
- note added: "* Espressif said ETA3485, SY8088 and RY3420 should also work, footprint looks the same (SOT23-5) * Waveshare also tested MP1605GTF-Z, Iq is only 11uA??? (lowest of all) but Espressif didn't say it work * ETA3485 and TLV62569 looks good to me"
- moved on the sheet: C35, C36, R2, R3, SW1, SW2
