File: power.kicad_sch (KiCad schematic)
At the start: 10 parts, among them U3 TLV62569DBV, U4 AP7361C-33E

Commit message: Finish off schematic
Other:
- note added: "* Espressif said ETA3485, SY8088 and RY3420 should also work, footprint looks the same (SOT23-5) * Waveshare also tested MP1605GTF-Z, Iq is only 11uA??? (lowest of all) but Espressif didn't say it work * ETA3485 and TLV62569 looks good to me"
- company: (none) -> By Jackson Ming Hu <huming2207@gmail.com> Copright (C) 2025 
- title: (none) -> Soul Probe
Changed lines of the file:
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@@
 	(generator_version "9.0")
 	(paper "A4")
+	(title_block
+		(title "Soul Probe")
+		(date "2025-11-28")
+		(rev "0.1")
+		(company "By Jackson Ming Hu <huming2207@gmail.com> Copright (C) 2025 ")
+		(comment 1 "Strictly no resell or commerical uses unless authorised by the author")
+	)
+	(text "* Espressif said ETA3485, SY8088 and RY3420 should also work, footprint looks the same (SOT23-5)\n* Waveshare also tested MP1605GTF-Z, Iq is only 11uA??? (lowest of all) but Espressif didn't say it work\n* ETA3485 and TLV62569 looks good to me"
+		(exclude_from_sim no)
+		(at 27.432 89.154 0)
+		(effects
+			(font
+				(size 1.27 1.27)
+			)
+			(justify left)
+		)
+	)
 	(text "5v to 3.3v LDO"
 		(exclude_from_sim no)
@@
 			)
 		)
-		(property "Description" ""
+		(property "Description" "Unpolarized capacitor, small symbol"
 			(at 166.37 55.88 0)
 			(effects
@@
 			)
 		)
-		(property "Description" ""
+		(property "Description" "Power symbol creates a global label with name \"+5V\""
 			(at 133.35 43.18 0)
 			(effects
@@
 			)
 		)
-		(property "Description" "C48945845"
+		(property "Description" "Inductor"
 			(at 74.93 44.45 0)
 			(effects
@@
 			)
 		)
-		(property "Description" ""
+		(property "Description" "Unpolarized capacitor, small symbol"
 			(at 176.53 55.88 0)
 			(effects
@@
 			)
 		)
-		(property "Description" ""
+		(property "Description" "Unpolarized capacitor, small symbol"
 			(at 143.51 55.88 0)
 			(effects
@@
 			)
 		)
-		(property "Description" ""
+		(property "Description" "Unpolarized capacitor, small symbol"
 			(at 133.35 55.88 0)
 			(effects
@@
 			)
 		)
-		(property "Description" ""
+		(property "Description" "Power symbol creates a global label with name \"GND\" , ground"
 			(at 157.48 62.23 0)
 			(effects

Commit message: Assign footprint
Parts:
- C1, C3, C37, C41: footprint Capacitor_SMD:C_0603_1608Metric -> Capacitor_SMD:C_0402_1005Metric
Changed lines of the file:
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@@
 			)
 		)
-		(property "Footprint" "Capacitor_SMD:C_0603_1608Metric"
+		(property "Footprint" "Capacitor_SMD:C_0402_1005Metric"
 			(at 32.7152 54.61 0)
 			(effects
@@
 			)
 		)
-		(property "Footprint" "Capacitor_SMD:C_0603_1608Metric"
+		(property "Footprint" "Capacitor_SMD:C_0402_1005Metric"
 			(at 176.53 55.88 0)
 			(effects
@@
 			)
 		)
-		(property "Footprint" "Capacitor_SMD:C_0603_1608Metric"
+		(property "Footprint" "Capacitor_SMD:C_0402_1005Metric"
 			(at 92.4052 53.34 0)
 			(effects
@@
 			)
 		)
-		(property "Footprint" "Capacitor_SMD:C_0603_1608Metric"
+		(property "Footprint" "Capacitor_SMD:C_0402_1005Metric"
 			(at 133.35 55.88 0)
 			(effects

Commit message: Rev 1
Parts:
- removed C1, C3: 22uF, Capacitor_SMD:C_0402_1005Metric, symbol Device:C
- removed C37, C41: 10uF, Capacitor_SMD:C_0402_1005Metric, symbol Device:C_Small
- removed C39, C40: 0.1uF, Capacitor_SMD:C_0402_1005Metric, symbol Device:C_Small
- removed JP1: 3V3PWR, Jumper:SolderJumper-2_P1.3mm_Bridged_Pad1.0x1.5mm, symbol Jumper:Jumper_2_Bridged
- removed L1: 2.2uH/3A, Inductor_SMD:L_Changjiang_FTC322510S, symbol Device:L
- removed U3: TLV62569DBV, Package_TO_SOT_SMD:SOT-23-5, symbol Regulator_Switching:TLV62569DBV
- removed U4: AP7361C-33E, Package_TO_SOT_SMD:SOT-223-3_TabPin2, symbol Regulator_Linear:AP7361C-33E
Other:
- note removed: "* Espressif said ETA3485, SY8088 and RY3420 should also work, footprint looks the same (SOT23-5) * Waveshare also tested MP1605GTF-Z, Iq is only 11uA??? (lowest of all) but Espressif didn't say it work * ETA3485 and TLV62569 looks good to me"
- note removed: "5v to 3.3v LDO"
