File: soulprobe.kicad_sch (KiCad schematic)
At the start: 0 parts

Commit message: Split schematic
Other:
- added sheet core (core.kicad_sch)
- added sheet peripheral (peripheral.kicad_sch)
- added sheet power (power.kicad_sch)
- note added: "* Espressif said ETA3485, SY8088 and RY3420 should also work, footprint looks the same (SOT23-5) * Waveshare also tested MP1605GTF-Z, Iq is only 11uA??? (lowest of all) but Espressif didn't say it work * ETA3485 and TLV62569 looks good to me"
- note added: "Simple ESP32-P4 Dev board By Jackson Ming Hu <huming2207@gmail.com> Copright (C) 2025"
Changed lines of the file:
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@@
 	(generator "eeschema")
 	(generator_version "9.0")
-	(paper "A4")
+	(paper "A3")
+	(text "* Espressif said ETA3485, SY8088 and RY3420 should also work, footprint looks the same (SOT23-5)\n* Waveshare also tested MP1605GTF-Z, Iq is only 11uA??? (lowest of all) but Espressif didn't say it work\n* ETA3485 and TLV62569 looks good to me"
+		(exclude_from_sim no)
+		(at 300.736 248.92 0)
+		(effects
+			(font
+				(size 1.27 1.27)
+			)
+			(justify left)
+		)
+	)
+	(text "Simple ESP32-P4 Dev board\nBy Jackson Ming Hu <huming2207@gmail.com>\nCopright (C) 2025 "
+		(exclude_from_sim no)
+		(at 309.372 260.858 0)
+		(effects
+			(font
+				(size 1.27 1.27)
+			)
+			(justify left)
+		)
+	)
+	(sheet
+		(at 121.92 134.62)
+		(size 36.83 26.67)
+		(exclude_from_sim no)
+		(in_bom yes)
+		(on_board yes)
+		(dnp no)
+		(fields_autoplaced yes)
+		(stroke
+			(width 0.1524)
+			(type solid)
+		)
+		(fill
+			(color 0 0 0 0.0000)
+		)
+		(property "Sheetname" "peripheral"
+			(at 121.92 133.9084 0)
+			(effects
+				(font
+					(size 1.27 1.27)
+				)
+				(justify left bottom)
+			)
+		)
+		(property "Sheetfile" "peripheral.kicad_sch"
+			(at 121.92 161.8746 0)
+			(effects
+				(font
+					(size 1.27 1.27)
+				)
+				(justify left top)
+			)
+		)
+		(instances
+			(project "soulprobe"
+				(path "/e5669c4b-5924-4e3d-8c50-ca267302db45"
+					(page "3")
+				)
+			)
+		)
+	)
+	(sheet
+		(at 173.99 134.62)
+		(size 45.72 26.67)
+		(exclude_from_sim no)
+		(in_bom yes)
+		(on_board yes)
+		(dnp no)
+		(fields_autoplaced yes)
+		(stroke
+			(width 0.1524)
+			(type solid)
+		)
+		(fill
+			(color 0 0 0 0.0000)
+		)
+		(property "Sheetname" "core"
+			(at 173.99 133.9084 0)
+			(effects
+				(font
+					(size 1.27 1.27)
+				)
+				(justify left bottom)
+			)
+		)
+		(property "Sheetfile" "core.kicad_sch"
+			(at 173.99 161.8746 0)
+			(effects
+				(font
+					(size 1.27 1.27)
+				)
+				(justify left top)
+			)
+		)
+		(instances
+			(project "soulprobe"
+				(path "/e5669c4b-5924-4e3d-8c50-ca267302db45"
+					(page "2")
+				)
+			)
+		)
+	)
+	(sheet
+		(at 68.58 134.62)
+		(size 35.56 26.67)
+		(exclude_from_sim no)
+		(in_bom yes)
+		(on_board yes)
+		(dnp no)
+		(fields_autoplaced yes)
+		(stroke
+			(width 0.1524)
+			(type solid)
+		)
+		(fill
+			(color 0 0 0 0.0000)
+		)
+		(property "Sheetname" "power"
+			(at 68.58 133.9084 0)
+			(effects
+				(font
+					(size 1.27 1.27)
+				)
+				(justify left bottom)
+			)
+		)
+		(property "Sheetfile" "power.kicad_sch"
+			(at 68.58 161.8746 0)
+			(effects
+				(font
+					(size 1.27 1.27)
+				)
+				(justify left top)
+			)
+		)
+		(instances
+			(project "soulprobe"
+				(path "/e5669c4b-5924-4e3d-8c50-ca267302db45"
+					(page "4")
+				)
+			)
+		)
+	)
 	(sheet_instances
 		(path "/"

Commit message: Finish off schematic
Other:
- note removed: "* Espressif said ETA3485, SY8088 and RY3420 should also work, footprint looks the same (SOT23-5) * Waveshare also tested MP1605GTF-Z, Iq is only 11uA??? (lowest of all) but Espressif didn't say it work * ETA3485 and TLV62569 looks good to me"
- note removed: "Simple ESP32-P4 Dev board By Jackson Ming Hu <huming2207@gmail.com> Copright (C) 2025"
- company: (none) -> By Jackson Ming Hu <huming2207@gmail.com> Copright (C) 2025 
- title: (none) -> Soul Probe
Changed lines of the file:
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@@
 	(generator "eeschema")
 	(generator_version "9.0")
-	(paper "A3")
-	(text "* Espressif said ETA3485, SY8088 and RY3420 should also work, footprint looks the same (SOT23-5)\n* Waveshare also tested MP1605GTF-Z, Iq is only 11uA??? (lowest of all) but Espressif didn't say it work\n* ETA3485 and TLV62569 looks good to me"
-		(exclude_from_sim no)
-		(at 300.736 248.92 0)
-		(effects
-			(font
-				(size 1.27 1.27)
-			)
-			(justify left)
-		)
-	)
-	(text "Simple ESP32-P4 Dev board\nBy Jackson Ming Hu <huming2207@gmail.com>\nCopright (C) 2025 "
-		(exclude_from_sim no)
-		(at 309.372 260.858 0)
-		(effects
-			(font
-				(size 1.27 1.27)
-			)
-			(justify left)
-		)
+	(paper "A4")
+	(title_block
+		(title "Soul Probe")
+		(date "2025-11-28")
+		(rev "0.1")
+		(company "By Jackson Ming Hu <huming2207@gmail.com> Copright (C) 2025 ")
+		(comment 1 "Strictly no resell or commerical uses unless authorised by the author")
 	)
 	(sheet
-		(at 121.92 134.62)
+		(at 120.65 68.58)
 		(size 36.83 26.67)
 		(exclude_from_sim no)
@@
 		)
 		(property "Sheetname" "peripheral"
-			(at 121.92 133.9084 0)
+			(at 120.65 67.8684 0)
 			(effects
 				(font
@@
 		)
 		(property "Sheetfile" "peripheral.kicad_sch"
-			(at 121.92 161.8746 0)
+			(at 120.65 95.8346 0)
 			(effects
 				(font
@@
 	)
 	(sheet
-		(at 173.99 134.62)
+		(at 172.72 68.58)
 		(size 45.72 26.67)
 		(exclude_from_sim no)
@@
 		)
 		(property "Sheetname" "core"
-			(at 173.99 133.9084 0)
+			(at 172.72 67.8684 0)
 			(effects
 				(font
@@
 		)
 		(property "Sheetfile" "core.kicad_sch"
-			(at 173.99 161.8746 0)
+			(at 172.72 95.8346 0)
 			(effects
 				(font
@@
 	)
 	(sheet
-		(at 68.58 134.62)
+		(at 67.31 68.58)
 		(size 35.56 26.67)
 		(exclude_from_sim no)
@@
 		)
 		(property "Sheetname" "power"
-			(at 68.58 133.9084 0)
+			(at 67.31 67.8684 0)
 			(effects
 				(font
@@
 		)
 		(property "Sheetfile" "power.kicad_sch"
-			(at 68.58 161.8746 0)
+			(at 67.31 95.8346 0)
 			(effects
 				(font

Commit message: Rev 1
Parts:
- added C1, C3: 22uF, Capacitor_SMD:C_0402_1005Metric, symbol Device:C
- added C10, C25: 20pF, Capacitor_SMD:C_0402_1005Metric, symbol Device:C
- added C11, C14, C20, C28: 10uF, Capacitor_SMD:C_0402_1005Metric, symbol Device:C
- added C12, C13, C15, C16, C21, C23, C24, C26, C29, C31, C33, C35, C36, C38, C6, C7, C8, C9: 0.1uF, Capacitor_SMD:C_0402_1005Metric, symbol Device:C
- added C17, C18, C19, C22, C27, C30: 1uF, Capacitor_SMD:C_0402_1005Metric, symbol Device:C
- added C32: 10nF, Capacitor_SMD:C_0402_1005Metric, symbol Device:C
- added C34: 4.7uF, Capacitor_SMD:C_0402_1005Metric, symbol Device:C
- added C4, C5: 22pF, Capacitor_SMD:C_0402_1005Metric, symbol Device:C
- added H1, H2, H3, H4: Mount, MountingHole:MountingHole_2.2mm_M2_Pad, symbol Mechanical:MountingHole_Pad
- added J1: PROG_PIN, Connector_PinHeader_1.27mm:PinHeader_2x10_P1.27mm_Vertical_SMD, symbol Connector_Generic:Conn_02x10_Odd_Even
- added J2: UART_PROG, Connector_PinHeader_1.27mm:PinHeader_1x06_P1.27mm_Vertical, symbol Connector:Conn_01x06_Pin
- added J3: DBG_PINS, Connector_PinHeader_1.27mm:PinHeader_2x10_P1.27mm_Vertical_SMD, symbol Connector_Generic:Conn_02x10_Odd_Even
- added J4: SD_PINS, Connector_PinHeader_1.27mm:PinHeader_2x10_P1.27mm_Vertical_SMD, symbol Connector_Generic:Conn_02x10_Odd_Even
- added J5: USB_DBG, Connector_PinSocket_1.27mm:PinSocket_1x04_P1.27mm_Vertical, symbol Connector:Conn_01x04_Pin
- added L1: 2.2uH/3A, Inductor_SMD:L_Changjiang_FTC322510S, symbol Device:L
- added R1, R11, R2, R3: 10k, Resistor_SMD:R_0402_1005Metric, symbol Device:R
- added U1: ESP32-P4, Espressif:ESP32-P4, symbol Espressif:ESP32-P4
- added U2: W25Q128JVS, Package_SO:SOIC-8_5.3x5.3mm_P1.27mm, symbol Memory_Flash:W25Q128JVS
- added U3: TLV62569DBV, Package_TO_SOT_SMD:SOT-23-5, symbol Regulator_Switching:TLV62569DBV
- added Y1: 40MHz 10ppm, Crystal:Crystal_SMD_2016-4Pin_2.0x1.6mm, symbol Device:Crystal_GND24
- added Y2: 32.768k, Crystal:Crystal_SMD_3215-2Pin_3.2x1.5mm, symbol Device:Crystal
Connections:
- new net: L1.1, U3.3 (SW)
- new net: R1.2, U1.68 (GPIO36)
- new net +1V2: C15.1, C28.1, C29.1, C3.1, C8.1, L1.2, U1.26 (VDD_HP_0), U1.76 (VDD_HP_2), U1.91 (VDD_HP_3)
- new net +3V3: C1.1, C11.1, C12.1, C13.1, C14.1, C16.1, C20.1, C21.1, C23.1, C24.2, C32.1, C33.1, C34.1, C6.1, C7.1, C9.1, J1.1 (Pin_1), J1.2 (Pin_2), J2.1 (Pin_1), J3.1 (Pin_1), J3.2 (Pin_2), J3.3 (Pin_3), J3.4 (Pin_4), J4.1 (Pin_1), J4.2 (Pin_2), J5.1 (Pin_1), R1.1, R2.1, R3.1, U1.101 (VDD_ANA), U1.102 (VDD_BAT), U1.21 (VDD_IO_0), U1.51 (VDD_USBPHY), U1.62 (VDD_IO_4), U1.75 (VDD_LDO), U1.77 (VDD_DCDCC), U1.85 (VDD_IO_5), U1.9 (VDD_LP), U1.96 (VDD_IO_6), U3.4 (VIN)
- new net CHIP_PU: C36.1, J2.4 (Pin_4), J3.5 (Pin_5), R2.2, U1.103 (CHIP_PU)
- new net EN_DCDC: U1.79 (EN_DCDC), U3.1 (EN)
- new net FB_DCDC: U1.78 (FB_DCDC), U3.5 (FB)
- new net FLASH_CK: U1.32 (FLASH_CK), U2.6 (CLK)
- new net FLASH_CS: R11.1, U1.27 (FLASH_CS), U2.1 (~{CS})
- new net FLASH_D: U1.33 (FLASH_D), U2.5 (DI/IO_{0})
- new net FLASH_HD: U1.31 (FLASH_HOLD), U2.7 (~{HOLD}/~{RESET}/IO_{3})
- new net FLASH_Q: U1.28 (FLASH_Q), U2.2 (DO/IO_{1})
- new net FLASH_WP: U1.29 (FLASH_WP), U2.3 (~{WP}/IO_{2})
- new net GND: C1.2, C10.1, C11.2, C12.2, C13.2, C14.2, C15.2, C16.2, C17.2, C18.2, C19.2, C20.2, C21.2, C22.2, C23.2, C24.1, C25.2, C26.2, C27.2, C28.2, C29.2, C3.2, C30.2, C31.2, C32.2, C33.2, C34.2, C35.2, C36.2, C38.2, C4.1, C5.2, C6.2, C7.2, C8.2, C9.2, H1.1, H2.1, H3.1, H4.1, J1.12 (Pin_12), J1.13 (Pin_13), J1.16 (Pin_16), J1.4 (Pin_4), J2.6 (Pin_6), J3.17 (Pin_17), J3.18 (Pin_18), J3.19 (Pin_19), J3.20 (Pin_20), J3.9 (Pin_9), J4.17 (Pin_17), J4.19 (Pin_19), J4.20 (Pin_20), J5.4 (Pin_4), U1.105 (GND), U2.4 (GND), U3.2 (GND), Y1.2, Y1.4
- new net IO0/LSE: C10.2, U1.104 (GPIO0/ADC), Y2.1
- new net IO10/TDO: J1.17 (Pin_17), U1.11 (GPIO10/ADC)
- new net IO11/nRST: J1.19 (Pin_19), U1.12 (GPIO11/ADC)
- new net IO12: J1.10 (Pin_10), U1.13 (GPIO12/ADC)
- new net IO13: J1.14 (Pin_14), U1.14 (GPIO13/ADC)
- new net IO14/UART_TX: J1.18 (Pin_18), U1.15 (GPIO14/ADC)
- new net IO15/UART_RX: J1.20 (Pin_20), U1.16 (GPIO15/ADC)
- new net IO1/LSE: C25.1, U1.1 (GPIO1/ADC), Y2.2
- new net IO2: J1.6 (Pin_6), U1.2 (GPIO2/ADC)
- new net IO26: J3.8 (Pin_8), U1.55 (GPIO26/ADC/USB)
- new net IO27: J3.6 (Pin_6), U1.56 (GPIO27/ADC/USB)
- new net IO3: J1.8 (Pin_8), U1.3 (GPIO3/ADC)
- new net IO35/BOOT: C35.1, J2.5 (Pin_5), J3.7 (Pin_7), R3.2, U1.66 (GPIO35)
- new net IO37/U0TXD: J2.2 (Pin_2), J3.13 (Pin_13), U1.69 (GPIO37)
- new net IO38/U0RXD: J2.3 (Pin_3), J3.11 (Pin_11), U1.70 (GPIO38)
- new net IO39/SDDAT0: J4.5 (Pin_5), U1.80 (GPIO39)
- new net IO40/SDDAT1: J4.7 (Pin_7), U1.81 (GPIO40)
- new net IO41/SDDAT2: J4.9 (Pin_9), U1.82 (GPIO41)
- new net IO42/SDDAT3: J4.11 (Pin_11), U1.83 (GPIO42)
- new net IO43/SDCLK: J4.13 (Pin_13), U1.84 (GPIO43)
- new net IO44/SDCMD: J4.15 (Pin_15), U1.86 (GPIO44)
- new net IO45/SDDET: J4.3 (Pin_3), U1.87 (GPIO45)
- new net IO46: J4.4 (Pin_4), U1.88 (GPIO46)
- new net IO47: J4.6 (Pin_6), U1.89 (GPIO47)
- new net IO48: J4.8 (Pin_8), U1.90 (GPIO48)
- new net IO49: J4.10 (Pin_10), U1.92 (GPIO49/ADC)
- new net IO4/TRST: J1.3 (Pin_3), U1.4 (GPIO4/ADC)
- new net IO50: J4.12 (Pin_12), U1.93 (GPIO50/ADC)
- new net IO51: J4.14 (Pin_14), U1.94 (GPIO51/ADC)
- new net IO52: J4.16 (Pin_16), U1.95 (GPIO52/ADC)
- new net IO53: J4.18 (Pin_18), U1.97 (GPIO53/ADC)
- new net IO5/TDI: J1.5 (Pin_5), U1.5 (GPIO5/ADC)
- new net IO6/SWDIO: J1.7 (Pin_7), U1.6 (GPIO6/ADC)
- new net IO7/SWCLK: J1.9 (Pin_9), U1.7 (GPIO7/ADC)
- new net IO8/BOOT: J1.11 (Pin_11), U1.8 (GPIO8/ADC)
- new net IO9/nRST: J1.15 (Pin_15), U1.10 (GPIO9/ADC)
- new net JTAG_D+: J3.10 (Pin_10), J5.3 (Pin_3), U1.53 (GPIO25/ADC/USB)
- new net JTAG_D-: J3.12 (Pin_12), J5.2 (Pin_2), U1.52 (GPIO24/ADC/USB)
- new net USB_D+: J3.14 (Pin_14), U1.50 (USB-DP)
- new net USB_D-: J3.16 (Pin_16), U1.49 (USB-DM)
- new net VDDO3: C19.1, U1.73 (VDDO_3)
- new net VDDO4: C22.1, U1.74 (VDDO_4)
- new net VDDO_FLASH: C17.1, C30.1, C31.1, C38.1, R11.2, U1.30 (VDD_FLASH_IO), U1.71 (VDDO_FLASH), U2.8 (VCC)
- new net VDDO_PSRAM: C18.1, C26.1, C27.1, U1.59 (VDD_PSRAM_0), U1.67 (VDD_PSRAM_1), U1.72 (VDDO_PSRAM)
- new net XTAL_N: C5.1, U1.99 (XTAL_N), Y1.3
- new net XTAL_P: C4.2, U1.100 (XTAL_P), Y1.1
- no-connect marks 0 -> 32
Other:
- removed sheet core
- removed sheet peripheral
- removed sheet power
- note added: "* CL=12.5pF"
- note added: "* CL=15pF"
- note added: "* Espressif said ETA3485, SY8088 and RY3420 should also work, footprint looks the same (SOT23-5) * Waveshare also tested MP1605GTF-Z, Iq is only 11uA??? (lowest of all) but Espressif didn't say it work * ETA3485 and TLV62569 looks good to me"
- note added: "* GPIO35 is BOOT pin"
- note added: "* VDD_IO0"
- note added: "* VDD_LP"
