File: core/soulcore.kicad_pcb (KiCad board)
At the start: 4 copper layers, 45 x 40 mm, 55 parts, among them J1 PROG_PIN, J2 UART_PROG, J3 DBG_PINS, J4 SD_PINS, J5 USB_DBG, U1 ESP32-P4, U2 W25Q128JVS, U3 TLV62569DBV, Y1 40MHz 10ppm, Y2 32.768k

Commit message: Rev 1.1
Parts:
- moved C9 2.59 mm to (128.0, 115.7), turned to 90 degrees
- moved C6 1.72 mm to (123.6, 117.2)
- moved C11 1.27 mm to (109.7, 111.9)
- moved J3 0.64 mm to (142.5, 120.0)
- moved C23 0.59 mm to (132.2, 125.2)
- moved C5 0.46 mm to (121.6, 113.1)
- moved C17 0.43 mm to (134.0, 122.6)
- moved C18 0.42 mm to (133.9, 121.5)
- moved C8 0.33 mm to (125.8, 114.8)
- moved Y1 0.33 mm to (121.8, 114.9)
- moved C4 0.33 mm to (119.6, 115.3)
- moved C16 0.16 mm to (132.0, 120.2)
- moved C15 0.13 mm to (132.0, 119.2)
Connections:
- J1 pad 12: GND -> IO13
- J1 pad 14: IO13 -> IO14/UART_TX
- J1 pad 16: GND -> IO15/UART_RX
- J1 pad 18: IO14/UART_TX -> IO16
- J1 pad 20: IO15/UART_RX -> IO17
- J3 pad 3: +3V3 -> IO29
- J3 pad 4: +3V3 -> IO28
- U1 pad 17: unconnected-(U1-GPIO16/ADC-Pad17) -> IO16
- U1 pad 18: unconnected-(U1-GPIO17/ADC-Pad18) -> IO17
- U1 pad 57: unconnected-(U1-GPIO28-Pad57) -> IO28
- U1 pad 58: unconnected-(U1-GPIO29-Pad58) -> IO29
Routing:
- net IO29: track 0.00 -> 21.3 mm, vias 0 -> 2
- net GND: track 39.0 -> 59.4 mm, vias 95 -> 103
- net IO28: track 0.00 -> 20.2 mm, vias 0 -> 2
- net +3V3: track 78.6 -> 61.7 mm, vias 24 -> 20
- net IO16: track 0.00 -> 15.5 mm, vias 0 -> 1
- net IO17: track 0.00 -> 15.1 mm, vias 0 -> 1
- net IO35/BOOT: track 33.7 -> 35.7 mm
- net +1V2: track 45.9 -> 47.5 mm, vias 4 -> 3
- net IO14/UART_TX: track 15.3 -> 16.7 mm
- net VDDO_FLASH: track 38.4 -> 39.7 mm
- net IO44/SDCMD: track 15.7 -> 14.4 mm
- net IO38/U0RXD: track 26.4 -> 27.6 mm
- net IO40/SDDAT1: track 13.2 -> 14.3 mm
- net IO41/SDDAT2: track 13.7 -> 14.7 mm
- net IO12: track 17.2 -> 18.2 mm
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Other:
- board text added: "SoulCore-ESP32P4 By Jackson M Hu Rev. 1.1 Jan 2026"
- board text removed: "SoulCore-ESP32P4 By Jackson M Hu Rev. 1 Dec 2025"
