File: core/soulcore.kicad_sch (KiCad schematic)
At the start: 55 parts, among them J1 PROG_PIN, J2 UART_PROG, J3 DBG_PINS, J4 SD_PINS, J5 USB_DBG, U1 ESP32-P4, U2 W25Q128JVS, U3 TLV62569DBV, Y1 40MHz 10ppm, Y2 32.768k

Commit message: Rev 1 - rename to soulcore
Parts:
- J2: footprint Connector_PinHeader_1.27mm:PinHeader_1x06_P1.27mm_Vertical -> Connector_PinSocket_2.00mm:PinSocket_1x06_P2.00mm_Vertical
- J5: footprint Connector_PinSocket_1.27mm:PinSocket_1x04_P1.27mm_Vertical -> Connector_PinSocket_2.00mm:PinSocket_1x04_P2.00mm_Vertical
Changed lines of the file:
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@@
 			)
 		)
-		(property "Footprint" "Connector_PinSocket_1.27mm:PinSocket_1x04_P1.27mm_Vertical"
+		(property "Footprint" "Connector_PinSocket_2.00mm:PinSocket_1x04_P2.00mm_Vertical"
 			(at 297.18 139.7 0)
 			(effects
@@
 			)
 		)
-		(property "Footprint" "Connector_PinHeader_1.27mm:PinHeader_1x06_P1.27mm_Vertical"
+		(property "Footprint" "Connector_PinSocket_2.00mm:PinSocket_1x06_P2.00mm_Vertical"
 			(at 374.65 142.24 0)
 			(effects

Commit message: Rev 1.1
Connections:
- net +3V3: no longer J3.3 (Pin_3), J3.4 (Pin_4)
- net GND: no longer J1.12 (Pin_12), J1.16 (Pin_16)
- net IO13: now also J1.12 (Pin_12); no longer J1.14 (Pin_14)
- net IO14/UART_TX: now also J1.14 (Pin_14); no longer J1.18 (Pin_18)
- net IO15/UART_RX: now also J1.16 (Pin_16); no longer J1.20 (Pin_20)
- net IO16: now reaches U1.17 (GPIO16/ADC)
- net IO16: now also J1.18 (Pin_18)
- net IO17: now reaches U1.18 (GPIO17/ADC)
- net IO17: now also J1.20 (Pin_20)
- net IO28: now reaches U1.57 (GPIO28)
- net IO28: now also J3.4 (Pin_4)
- net IO29: now reaches U1.58 (GPIO29)
- net IO29: now also J3.3 (Pin_3)
- no-connect marks 32 -> 28
